File: 2x2 micro pad.kicad_pcb (KiCad board)
At the start: 2 copper layers, 69.8 x 38.1 mm, 24 parts, among them SW1 SW_Push, U1 ATmega32U4-AU, Y1 16MHz

Commit message: pcb 2
Parts:
- C4, C5, C6, C7, F1, R2, R3, SW1, USB1: moved to B.Cu
- moved R2 69.3 mm to (176.2, 67.5), turned to 90 degrees
- moved SW1 68.9 mm to (172.2, 89.7)
- moved USB1 59.5 mm to (173.8, 57.1), turned to 270 degrees
- moved R3 55.6 mm to (173.0, 67.5), turned to 270 degrees
- moved C4 52.9 mm to (181.8, 58.7), turned to 270 degrees
- moved C7 43.9 mm to (186.5, 58.7), turned to 270 degrees
- moved F1 43.2 mm to (169.9, 66.7), turned to 90 degrees
- moved C6 35.3 mm to (189.7, 58.7), turned to 270 degrees
- moved C5 29.0 mm to (193.7, 58.7), turned to 270 degrees
- moved C3 16.8 mm to (181.0, 91.3), turned to 0 degrees
- moved C1 9.26 mm to (180.8, 69.7)
- moved C2 9.26 mm to (191.1, 69.7)
- moved Y1 9.26 mm to (185.6, 69.7)
- moved R4 8.97 mm to (190.5, 91.3)
- moved R1 7.02 mm to (196.1, 74.6), turned to 90 degrees
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Other:
- outline, holes or cut-outs redrawn

Commit message: pcb routing
Parts:
- moved C6 30.3 mm to (169.1, 81.0)
- moved C5 29.8 mm to (173.8, 81.0)
- moved C4 24.5 mm to (171.4, 81.0)
- moved C7 24.5 mm to (176.2, 81.0)
- moved C1 5.08 mm to (182.6, 64.9)
- moved Y1 5.02 mm to (187.2, 64.9)
- moved U1 4.83 mm to (186.5, 76.2)
- moved C2 4.77 mm to (191.3, 64.9)
- moved C3 2.25 mm to (182.6, 89.7)
- moved F1 1.77 mm to (169.1, 68.3)
- moved R2 1.59 mm to (174.6, 67.5)
- moved R4 1.59 mm to (190.5, 89.7)
- moved R1 0.79 mm to (196.1, 73.8)
- moved R3 0.79 mm to (172.2, 67.5), turned to 90 degrees
Connections:
- U1 pad 29: Net-(U1-Pad29) -> COL1
- U1 pad 30: Net-(U1-Pad30) -> COL0
- U1 pad 31: Net-(U1-Pad31) -> ROW0
- U1 pad 32: Net-(U1-Pad32) -> ROW1
Routing:
- net GND: track 0.00 -> 116.3 mm, vias 0 -> 2
- net +5V: track 0.00 -> 101.1 mm, vias 0 -> 4
- net COL1: track 0.00 -> 66.5 mm
- net Net-(R1-Pad2): track 0.00 -> 51.2 mm, vias 0 -> 3
- net ROW0: track 0.00 -> 48.6 mm
- net ROW1: track 0.00 -> 48.1 mm
- net COL0: track 0.00 -> 41.8 mm
- net Net-(C1-Pad1): track 0.00 -> 24.5 mm
- net Net-(C3-Pad1): track 0.00 -> 19.4 mm, vias 0 -> 2
- net Net-(R3-Pad1): track 0.00 -> 15.5 mm
- net Net-(R2-Pad1): track 0.00 -> 12.8 mm
- net Net-(R4-Pad2): track 0.00 -> 9.82 mm
- net Net-(C2-Pad1): track 0.00 -> 8.87 mm
- net Net-(D1-Pad2): track 0.00 -> 6.82 mm
- net Net-(D2-Pad2): track 0.00 -> 6.82 mm
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Other:
- net class Default: trace_width 0.25 -> 0.254
- net class power added: clearance 0.2, trace_width 0.381, via_dia 0.8, via_drill 0.4

Commit message: pcb update
Parts:
- added G***: LOGO, LOGO:juhua1, F.Cu at (188.0, 86.4)
Routing:
- added copper zone on B.Cu, net GND
Other:
- board text added: "Dreammaker"
